Commit message: main

File: luminous_description/urdf/luminous_description.xacro (robot description, xacro)
@@ -1,5 +1,4 @@
 <?xml version="1.0" encoding="utf-8"?>
 <robot name="luminous_description" xmlns:xacro="http://www.ros.org/wiki/xacro">
-<xacro:include filename="$(find realsense2_description)/urdf/_d435.urdf.xacro" />
 <xacro:macro name="luminous_description" params="footprint_link:=true">
   <xacro:if value="${footprint_link}">
@@ -597,7 +596,4 @@
   <axis xyz="0 0 0" />
 </joint>
-<xacro:sensor_d435 name="camera" topics_ns="camera" parent="base_link" publish_pointcloud="true">
-    <origin xyz="0.060893 -0.22847 -0.029728" rpy="0 0 0" />
-  </xacro:sensor_d435>
 <!-- ######################################################################################### -->
   <transmission name="front_right_wheel_trans" type="SimpleTransmission">
